File: ws2812.kicad_pcb (KiCad board)
At the start: 2 copper layers, 88 x 40 mm, 137 parts, among them J1 X_WF-04S, Q1 IRLML2502

Commit message: sablono failu paruosimas
Parts:
- added REF**: SolderWirePad_single_0-8mmDrill, Wire_Pads:SolderWirePad_single_0-8mmDrill, F.Cu at (88.7, 118.0)
- added REF**: SolderWirePad_single_0-8mmDrill, Wire_Pads:SolderWirePad_single_0-8mmDrill, F.Cu at (158.6, 106.7)
- added REF**: SolderWirePad_single_0-8mmDrill, Wire_Pads:SolderWirePad_single_0-8mmDrill, F.Cu at (158.5, 98.6)
- added REF**: SolderWirePad_single_0-8mmDrill, Wire_Pads:SolderWirePad_single_0-8mmDrill, F.Cu at (88.7, 110.0)
- added REF**: SolderWirePad_single_0-8mmDrill, Wire_Pads:SolderWirePad_single_0-8mmDrill, F.Cu at (88.6, 102.0)
- added REF**: SolderWirePad_single_0-8mmDrill, Wire_Pads:SolderWirePad_single_0-8mmDrill, F.Cu at (160.6, 90.5)
Routing:
- net /DATA1: track 81.8 -> 3.82 mm, vias 2 -> 0
- net /DATA3: track 81.4 -> 4.48 mm, vias 2 -> 0
- net /DATA2: track 81.3 -> 5.16 mm, vias 2 -> 0
- net VCC: track 444.4 -> 445.1 mm
Other:
- net class Default: clearance 0.3 -> 0.25
- rule trace_clearance: 0.3 -> 0.25
- board text added: "WS2812"
